File: pcb/qqv11.sch (KiCad schematic (older format))
At the start: 107 parts, among them J1 Conn_02x04_Odd_Even, J2 VCQQV1OP, J3 Conn_02x07_Odd_Even, J4 10118194-0001LF, J5 Conn_01x06, J6 Conn_02x02_Odd_Even, J7 Conn_01x03, Q1 AON7804, Q2 AON7804, Q3 AON7423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

Commit message: added pictures
Parts:
- MK1: symbol CMC-4015-40P:CMC-4015-40P -> qqv11-rescue:CMC-4015-40P-CMC-4015-40P
Other:
- moved on the sheet: A1
Changed lines of the file:
@@
 Wire Wire Line
 	16050 10600 15650 10600
-Text Label 1300 5300 0    50   ~ 0
+Text Label 1250 4550 0    50   ~ 0
 I-~RST~
-Text Label 2800 5200 2    50   ~ 0
+Text Label 2750 4450 2    50   ~ 0
 I-INT
 Wire Wire Line
@@
 Wire Wire Line
 	9200 1900 9200 2000
-Text Label 2800 5400 2    50   ~ 0
+Text Label 2750 4650 2    50   ~ 0
 I-RX
-Text Label 2800 5300 2    50   ~ 0
+Text Label 2750 4550 2    50   ~ 0
 I-TX
 $Comp
@@
 	7550 3050 7550 3150
 $Comp
-L CMC-4015-40P:CMC-4015-40P MK1
+L qqv11-rescue:CMC-4015-40P-CMC-4015-40P MK1
 U 1 1 5D389BE9
 P 1050 2750
@@
 L vc_conn:vc_bosch_imu_pcb A1
 U 1 1 5D7034BF
-P 2050 5350
-F 0 "A1" H 2050 5725 50  0000 C CNN
-F 1 "vc_bosch_imu_pcb" H 2050 5634 50  0000 C CNN
-F 2 "VC:VC_bosch_imu_pcb_mod" H 2050 5350 50  0001 C CNN
-F 3 "" H 2050 5350 50  0001 C CNN
-	1    2050 5350
+P 2000 4600
+F 0 "A1" H 2000 4975 50  0000 C CNN
+F 1 "vc_bosch_imu_pcb" H 2000 4884 50  0000 C CNN
+F 2 "VC:VC_bosch_imu_pcb_mod" H 2000 4600 50  0001 C CNN
+F 3 "" H 2000 4600 50  0001 C CNN
+	1    2000 4600
 	1    0    0    -1
 $EndComp
@@
 L power:+3.3V #PWR045
 U 1 1 5D75B16A
-P 1500 5150
-F 0 "#PWR045" H 1500 5000 50  0001 C CNN
-F 1 "+3.3V" H 1515 5323 50  0000 C CNN
-F 2 "" H 1500 5150 50  0001 C CNN
-F 3 "" H 1500 5150 50  0001 C CNN
-	1    1500 5150
+P 1450 4400
+F 0 "#PWR045" H 1450 4250 50  0001 C CNN
+F 1 "+3.3V" H 1465 4573 50  0000 C CNN
+F 2 "" H 1450 4400 50  0001 C CNN
+F 3 "" H 1450 4400 50  0001 C CNN
+	1    1450 4400
 	1    0    0    -1
 $EndComp
@@
 L power:GND #PWR051
 U 1 1 5D75BE10
-P 1500 5550
-F 0 "#PWR051" H 1500 5300 50  0001 C CNN
-F 1 "GND" H 1505 5377 50  0000 C CNN
-F 2 "" H 1500 5550 50  0001 C CNN
-F 3 "" H 1500 5550 50  0001 C CNN
-	1    1500 5550
-	1    0    0    -1
-$EndComp
-Wire Wire Line
-	1500 5200 1600 5200
-Wire Wire Line
-	1500 5150 1500 5200
-Wire Wire Line
-	1600 5500 1500 5500
-Wire Wire Line
-	1500 5500 1500 5550
-Wire Wire Line
-	1300 5300 1600 5300
-Wire Wire Line
-	1300 5400 1600 5400
-Wire Wire Line
-	2800 5200 2500 5200
-Text Label 1300 5400 0    50   ~ 0
+P 1450 4800
+F 0 "#PWR051" H 1450 4550 50  0001 C CNN
+F 1 "GND" H 1455 4627 50  0000 C CNN
+F 2 "" H 1450 4800 50  0001 C CNN
+F 3 "" H 1450 4800 50  0001 C CNN
+	1    1450 4800
+	1    0    0    -1
+$EndComp
+Wire Wire Line
+	1450 4450 1550 4450
+Wire Wire Line
+	1450 4400 1450 4450
+Wire Wire Line
+	1550 4750 1450 4750
+Wire Wire Line
+	1450 4750 1450 4800
+Wire Wire Line
+	1250 4550 1550 4550
+Wire Wire Line
+	1250 4650 1550 4650
+Wire Wire Line
+	2750 4450 2450 4450
+Text Label 1250 4650 0    50   ~ 0
 I-~BOOT~
 Wire Wire Line
-	2800 5300 2500 5300
-Wire Wire Line
-	2800 5400 2500 5400
+	2750 4550 2450 4550
+Wire Wire Line
+	2750 4650 2450 4650
 $Comp
 L power:GND #PWR052
 U 1 1 5DB4CB73
-P 2600 5550
-F 0 "#PWR052" H 2600 5300 50  0001 C CNN
-F 1 "GND" H 2605 5377 50  0000 C CNN
-F 2 "" H 2600 5550 50  0001 C CNN
-F 3 "" H 2600 5550 50  0001 C CNN
-	1    2600 5550
-	1    0    0    -1
-$EndComp
-Wire Wire Line
-	2500 5500 2600 5500
-Wire Wire Line
-	2600 5500 2600 5550
+P 2550 4800
+F 0 "#PWR052" H 2550 4550 50  0001 C CNN
+F 1 "GND" H 2555 4627 50  0000 C CNN
+F 2 "" H 2550 4800 50  0001 C CNN
+F 3 "" H 2550 4800 50  0001 C CNN
+	1    2550 4800
+	1    0    0    -1
+$EndComp
+Wire Wire Line
+	2450 4750 2550 4750
+Wire Wire Line
+	2550 4750 2550 4800
 $Comp
 L RF_Module:ESP32-WROOM-32D U8

Commit message: revised
Other:
- note added: "ADD resistor to avoid problems when programing"
- note added: "ERROR, need correction, when using secondary oscilator connect de clock signal to SOSCO no SOSCI\n"
Changed lines of the file:
@@
 	1    0    0    -1
 $EndComp
+Text Notes 9950 5250 0    50   Italic 10
+ERROR, need correction,  when using secondary oscilator connect de clock signal to SOSCO no SOSCI\n
+Text Notes 6450 12650 0    50   ~ 0
+ADD resistor to avoid problems when programing
 $EndSCHEMATC
